File: eagle/board/ControlBoard.sch (EAGLE design)
At the start: 18 parts, among them CN1 PIC_CN_H, J1 TB112-2-2-U-1, J2 TB112-2-2-U-1, Q1 IN-12B, Q2 IN-12B, SW1 10-XX, U1 TLP627-2, U2 SN74141, U3 PIC16F1823-I/P, X1 20MHz

Commit message: 点灯制御の回路図を修正
PICのVDDが5Vにつながっていなかったので修正
Connections:
- removed net N$3: C1.2, U3.VDD
- net +5V: now also C1.2, U3.VDD
Changed lines of the file:
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@@
 <part name="CN1" library="Connectors" deviceset="PIC_CN" device="_H"/>
 <part name="P+1" library="Supply" deviceset="+5V" device=""/>
-<part name="P+2" library="Supply" deviceset="+5V" device=""/>
 <part name="P+3" library="Supply" deviceset="+170V" device=""/>
 <part name="GND2" library="Supply" deviceset="0V" device=""/>
@@
 <instance part="CN1" gate="G$1" x="109.22" y="114.3"/>
 <instance part="P+1" gate="1" x="175.26" y="88.9"/>
-<instance part="P+2" gate="1" x="101.6" y="134.62"/>
 <instance part="P+3" gate="1" x="139.7" y="106.68"/>
 <instance part="GND2" gate="1" x="106.68" y="43.18"/>
@@
 </segment>
 <segment>
-<pinref part="P+2" gate="1" pin="+5V"/>
-<wire x1="101.6" y1="132.08" x2="101.6" y2="116.84" width="0.1524" layer="91"/>
 <pinref part="CN1" gate="G$1" pin="VDD"/>
-<wire x1="101.6" y1="116.84" x2="109.22" y2="116.84" width="0.1524" layer="91"/>
-</segment>
-<segment>
+<wire x1="109.22" y1="116.84" x2="81.28" y2="116.84" width="0.1524" layer="91"/>
+<wire x1="81.28" y1="116.84" x2="81.28" y2="104.14" width="0.1524" layer="91"/>
+<wire x1="81.28" y1="104.14" x2="33.02" y2="104.14" width="0.1524" layer="91"/>
+<wire x1="33.02" y1="104.14" x2="33.02" y2="78.74" width="0.1524" layer="91"/>
+<pinref part="U3" gate="G$1" pin="VDD"/>
+<wire x1="43.18" y1="78.74" x2="38.1" y2="78.74" width="0.1524" layer="91"/>
+<pinref part="C1" gate="G$1" pin="2"/>
+<wire x1="38.1" y1="78.74" x2="38.1" y2="83.82" width="0.1524" layer="91"/>
+<wire x1="33.02" y1="78.74" x2="38.1" y2="78.74" width="0.1524" layer="91"/>
+<junction x="38.1" y="78.74"/>
 <pinref part="P+4" gate="1" pin="+5V"/>
 <wire x1="27.94" y1="132.08" x2="27.94" y2="127" width="0.1524" layer="91"/>
 <pinref part="J1" gate="G$1" pin="1"/>
-<wire x1="27.94" y1="127" x2="55.88" y2="127" width="0.1524" layer="91"/>
+<wire x1="27.94" y1="127" x2="33.02" y2="127" width="0.1524" layer="91"/>
 <pinref part="R3" gate="G$1" pin="2"/>
+<wire x1="33.02" y1="127" x2="55.88" y2="127" width="0.1524" layer="91"/>
 <wire x1="27.94" y1="119.38" x2="27.94" y2="127" width="0.1524" layer="91"/>
 <junction x="27.94" y="127"/>
+<wire x1="33.02" y1="104.14" x2="33.02" y2="127" width="0.1524" layer="91"/>
+<junction x="33.02" y="104.14"/>
+<junction x="33.02" y="127"/>
 </segment>
 </net>
@@
 </segment>
 </net>
-<net name="N$3" class="0">
-<segment>
-<pinref part="U3" gate="G$1" pin="VDD"/>
-<wire x1="43.18" y1="78.74" x2="38.1" y2="78.74" width="0.1524" layer="91"/>
-<pinref part="C1" gate="G$1" pin="2"/>
-<wire x1="38.1" y1="78.74" x2="38.1" y2="83.82" width="0.1524" layer="91"/>
-</segment>
-</net>
