File: eagle/board/DigitDisplayBoard.sch (EAGLE design)
At the start: 43 parts, among them CN1 PIC_CN_H, J1 2DC0005D1000, Q1 2SA1020L-Y, Q2 2SK3234, Q3 IN-12B, Q4 IN-12B, Q5 IN-12B, SW1 10-XX, U1 MC34063AP1, U2 SN74141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

Commit message: ３桁表示用基板の使用部品を修正
ライブラリーを修正（抵抗器）
基板で使用する部品の見直し
Parts:
- C7, C8: device Parts:CAP_100MIL -> Parts:CAP_200MIL
- R10, R11, R12, R13, R14, R15, R8: device Parts:RESISTOR_600MIL -> Parts:RESISTOR_300MIL
Changed lines of the file:
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@@
 <part name="U3" library="Parts" deviceset="TLP627*" device="-2"/>
 <part name="C9" library="Parts" deviceset="CAP" device="_200MIL" value="0.1uF"/>
-<part name="R8" library="Parts" deviceset="RESISTOR" device="_600MIL" value="20k"/>
+<part name="R8" library="Parts" deviceset="RESISTOR" device="_300MIL" value="20k"/>
 <part name="R9" library="Parts" deviceset="RESISTOR" device="_600MIL" value="20k"/>
-<part name="R15" library="Parts" deviceset="RESISTOR" device="_600MIL" value="10k"/>
-<part name="R11" library="Parts" deviceset="RESISTOR" device="_600MIL" value="470"/>
-<part name="R12" library="Parts" deviceset="RESISTOR" device="_600MIL" value="470"/>
+<part name="R15" library="Parts" deviceset="RESISTOR" device="_300MIL" value="10k"/>
+<part name="R11" library="Parts" deviceset="RESISTOR" device="_300MIL" value="470"/>
+<part name="R12" library="Parts" deviceset="RESISTOR" device="_300MIL" value="470"/>
 <part name="GND2" library="Supply" deviceset="0V" device=""/>
 <part name="CN1" library="Connectors" deviceset="PIC_CN" device="_H"/>
@@
 <part name="GND4" library="Supply" deviceset="0V" device=""/>
 <part name="GND5" library="Supply" deviceset="0V" device=""/>
-<part name="C7" library="Parts" deviceset="CAP" device="_100MIL" value="22pF"/>
-<part name="C8" library="Parts" deviceset="CAP" device="_100MIL" value="22pF"/>
+<part name="C7" library="Parts" deviceset="CAP" device="_200MIL" value="22pF"/>
+<part name="C8" library="Parts" deviceset="CAP" device="_200MIL" value="22pF"/>
 <part name="P+5" library="Supply" deviceset="+5V" device=""/>
 <part name="GND8" library="Supply" deviceset="0V" device=""/>
@@
 <part name="GND6" library="Supply" deviceset="0V" device=""/>
 <part name="U4" library="Parts" deviceset="TLP627*" device="-2"/>
-<part name="R10" library="Parts" deviceset="RESISTOR" device="_600MIL" value="20k"/>
-<part name="R13" library="Parts" deviceset="RESISTOR" device="_600MIL" value="470"/>
-<part name="R14" library="Parts" deviceset="RESISTOR" device="_600MIL" value="470"/>
+<part name="R10" library="Parts" deviceset="RESISTOR" device="_300MIL" value="20k"/>
+<part name="R13" library="Parts" deviceset="RESISTOR" device="_300MIL" value="470"/>
+<part name="R14" library="Parts" deviceset="RESISTOR" device="_300MIL" value="470"/>
 <part name="P+8" library="Supply" deviceset="+170V" device=""/>
 <part name="GND7" library="Supply" deviceset="0V" device=""/>
